File: dats-kontrol-1kw-sysmin.kicad_pcb (KiCad board)
At the start: 2 copper layers, 26 parts, among them J1 SWD, J2 Conn_01x12, J3 USB_B, SW1 SW?, U1 AMS1117CD-3.3, U2 STM32F4X1CXU6, Y1 25MHZ 9PF, Y2 32.768KHz

Commit message: new layout
Parts:
- removed C1: 10uF, Capacitor_SMD:C_0805_2012Metric
- removed C10, C11, C12, C9: 100nF, Capacitor_SMD:C_0805_2012Metric
- removed C13: 100 nF, Capacitor_SMD:C_0805_2012Metric
- removed C2, C3: 12pF, Capacitor_SMD:C_0805_2012Metric
- removed C4, C5, C8: 4.3pF, Capacitor_SMD:C_0805_2012Metric
- removed C6: 10 uF, Capacitor_SMD:CP_Elec_5x5.3
- removed C7: 22 uF, Capacitor_SMD:C_0805_2012Metric
- removed D1: LED, LED_SMD:LED_0805_2012Metric
- removed H1, H2: M3_MH, MountingHole:MountingHole_3.2mm_M3
- removed J1: SWD, Connector_PinHeader_2.54mm:PinHeader_1x04_P2.54mm_Vertical
- removed J2: Conn_01x12, Connector_PinHeader_2.54mm:PinHeader_1x12_P2.54mm_Vertical
- removed J3: USB_B, Connector_USB:USB_B_TE_5787834_Vertical
- removed R1: 10, Resistor_SMD:R_0805_2012Metric
- removed R2: 10K, Resistor_SMD:R_0805_2012Metric
- removed SW1: SW?, Button_Switch_SMD:SW_Push_1P1T_NO_CK_KMR2
- removed U1: AMS1117CD-3.3, Package_TO_SOT_SMD:SOT-223-3_TabPin2
- removed U2: STM32F4X1CXU6, Package_DFN_QFN:QFN-48-1EP_7x7mm_P0.5mm_EP5.6x5.6mm
- removed Y1: 25MHZ 9PF, Crystal:Crystal_SMD_3225-4Pin_3.2x2.5mm_HandSoldering
- removed Y2: 32.768KHz, Crystal:Crystal_SMD_SeikoEpson_MC146-4Pin_6.7x1.5mm_HandSoldering
- added ?: , , F.Cu at (187.9, 70.8)
- added ?: , , F.Cu at (107.7, 99.8)
- added ?: MountingHole_3.2mm_M3, MountingHole:MountingHole_3.2mm_M3, F.Cu at (105.9, 78.3)
- added ?: MountingHole_3.2mm_M3, MountingHole:MountingHole_3.2mm_M3, F.Cu at (197.9, 142.2)
- added ?: MountingHole_3.2mm_M3, MountingHole:MountingHole_3.2mm_M3, F.Cu at (197.9, 78.3)
- added ?: , , F.Cu at (127.9, 70.8)
- added ?: , , F.Cu at (157.9, 70.8)
- added ?: MountingHole_3.2mm_M3, MountingHole:MountingHole_3.2mm_M3, F.Cu at (105.9, 142.2)
- added ?: , , F.Cu at (197.9, 142.2)
- added ?: , , F.Cu at (107.7, 109.7)
- added J10: PHASE_C_ISENSE, Connector_PinSocket_2.54mm:PinSocket_1x03_P2.54mm_Vertical, F.Cu at (171.9, 69.8)
- added J7: Conn_01x12, Connector_PinHeader_2.54mm:PinHeader_2x06_P2.54mm_Vertical, F.Cu at (107.5, 122.9)
- added J8: PHASE_A_ISENSE, Connector_PinSocket_2.54mm:PinSocket_1x03_P2.54mm_Vertical, F.Cu at (111.9, 69.8)
- added J9: PHASE_B_ISENSE, Connector_PinSocket_2.54mm:PinSocket_1x03_P2.54mm_Vertical, F.Cu at (141.9, 69.8)
Other:
- board outline added: 119.6 x 85 mm

Commit message: adding stm32 symbol+footprint
Parts:
- added U1: YAAJ_WeAct_BlackPill_Part_Like_SWD_Breakout, blackpill:YAAJ_WeAct_BlackPill_2, F.Cu at (133.6, 118.2)
- J10, J8, J9: footprint Connector_PinSocket_2.54mm:PinSocket_1x03_P2.54mm_Vertical -> Connector_PinHeader_2.54mm:PinHeader_1x03_P2.54mm_Vertical
Other:
- board size 119.6 x 85 mm -> 101 x 85.3 mm

Commit message: Layout STM
Parts:
- added C1: C, Resistor_SMD:R_0805_2012Metric, F.Cu at (172.2, 129.0)
- added J5: Conn_01x05, Connector_JST:JST_XH_B5B-XH-A_1x05_P2.50mm_Vertical, F.Cu at (125.0, 143.5)
- added J6: Conn_01x03, Connector_JST:JST_XH_B3B-XH-A_1x03_P2.50mm_Vertical, F.Cu at (150.6, 143.5)
- added J7: Conn_01x02, Connector_JST:JST_XH_B2B-XH-A_1x02_P2.50mm_Vertical, F.Cu at (171.2, 143.0)
- added R1: 10K, Resistor_SMD:R_0805_2012Metric, F.Cu at (125.9, 129.3)
- added R2: 10K, Resistor_SMD:R_0805_2012Metric, F.Cu at (128.4, 133.6)
- added R3: 10K, Resistor_SMD:R_0805_2012Metric, F.Cu at (130.9, 137.9)
- added R4: 1K, Resistor_SMD:R_0805_2012Metric, F.Cu at (172.2, 132.3)
- added R5: 120, Resistor_SMD:R_0805_2012Metric, F.Cu at (172.2, 135.6)
- added U2: MCP2551-I-SN, Package_SO:SOIC-8_3.9x4.9mm_P1.27mm, F.Cu at (163.4, 133.2)
- J1: renamed from J10; value PHASE_C_ISENSE -> Conn_01x03
- J2: renamed from J9; value PHASE_B_ISENSE -> Conn_01x03
- J3: renamed from J8; value PHASE_A_ISENSE -> Conn_01x03
- renumbered J7 to J4
Connections:
- J1 pad 1: (no net) -> +3V3
- J1 pad 2: (no net) -> CURRENT_SENS_C
- J1 pad 3: (no net) -> GND
- J2 pad 1: (no net) -> +3V3
- J2 pad 2: (no net) -> CURRENT_SENS_B
- J2 pad 3: (no net) -> GND
- J3 pad 1: (no net) -> +3V3
- J3 pad 2: (no net) -> CURRENT_SENS_A
- J3 pad 3: (no net) -> GND
- J4 pad 1: (no net) -> +3V3
- J4 pad 10: (no net) -> +3V3
- J4 pad 11: (no net) -> GND
- J4 pad 12: (no net) -> GND
- J4 pad 2: (no net) -> +3V3
- J4 pad 3: (no net) -> A_H
- J4 pad 4: (no net) -> A_L
- J4 pad 5: (no net) -> B_H
- J4 pad 6: (no net) -> B_L
- J4 pad 7: (no net) -> C_H
- J4 pad 8: (no net) -> C_L
- J4 pad 9: (no net) -> +3V3
- U1 pad 10: unconnected-(U1-PA15-Pad10) -> CAN_TX
- U1 pad 11: unconnected-(U1-PB3-Pad11) -> CAN_RX
- U1 pad 12: unconnected-(U1-PB4-Pad12) -> HALL_A
- U1 pad 13: unconnected-(U1-PB5-Pad13) -> HALL_B
- U1 pad 14: unconnected-(U1-PB6-Pad14) -> HALL_C
- U1 pad 19: unconnected-(U1-GND-Pad19) -> GND
- U1 pad 2: unconnected-(U1-PB13-Pad2) -> A_L
- U1 pad 20: unconnected-(U1-3V3-Pad20) -> +3V3
- U1 pad 3: unconnected-(U1-PB14-Pad3) -> B_L
- U1 pad 30: unconnected-(U1-PA4-Pad30) -> CURRENT_SENS_C
- U1 pad 31: unconnected-(U1-PA5-Pad31) -> THROTTLE
- U1 pad 34: unconnected-(U1-PB0-Pad34) -> CURRENT_SENS_A
- U1 pad 35: unconnected-(U1-PB1-Pad35) -> CURRENT_SENS_B
- U1 pad 38: unconnected-(U1-3V3-Pad38) -> +3V3
- U1 pad 39: unconnected-(U1-GND-Pad39) -> GND
- U1 pad 4: unconnected-(U1-PB15-Pad4) -> C_L
- U1 pad 40: unconnected-(U1-5V-Pad40) -> +5V
- U1 pad 5: unconnected-(U1-PA8-Pad5) -> A_H
- U1 pad 6: unconnected-(U1-PA9-Pad6) -> B_H
- U1 pad 7: unconnected-(U1-PA10-Pad7) -> C_H
Routing:
- net THROTTLE: track 0.00 -> 103.9 mm, vias 0 -> 1
- net CAN_TX: track 0.00 -> 76.4 mm
- net CAN_RX: track 0.00 -> 68.8 mm
- net C_H: track 0.00 -> 67.3 mm
- net CURRENT_SENS_A: track 0.00 -> 65.8 mm
- net B_H: track 0.00 -> 58.9 mm
- net HALL_A: track 0.00 -> 56.4 mm
- net HALL_B: track 0.00 -> 53.6 mm
- net HALL_C: track 0.00 -> 51.1 mm
- net A_H: track 0.00 -> 50.7 mm
- net CURRENT_SENS_C: track 0.00 -> 44.7 mm
- net C_L: track 0.00 -> 36.7 mm
- net CURRENT_SENS_B: track 0.00 -> 34.0 mm
- net B_L: track 0.00 -> 32.9 mm
- net A_L: track 0.00 -> 29.3 mm
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- added copper zone on B.Cu, net +3V3
- added copper zone on F.Cu, net +3V3
- added copper zone on B.Cu, net +5V
- added copper zone on F.Cu, net +5V
- added copper zone on B.Cu, net GND
- added copper zone on F.Cu, net GND

Commit message: adding some background
Parts:
- added G***: LOGO, symbols:modrive_16mm, F.Cu at (156.3, 89.8)
Routing:
- net CURRENT_SENS_A: track 65.8 -> 68.9 mm
- net GND: vias 55 -> 33
- net +5V: vias 10 -> 3
- net +3V3: vias 21 -> 12
Other:
- outline, holes or cut-outs redrawn
- board text added: "CAN BUS"
- board text added: "HALL IN"
- board text added: "THRL IN"
